Commit message: feat(kinematics): integrate neck joint, realign neck_link_2 visuals, attach camera_1 to neck_link_2, and add missing joints to ros2_control

File: vectorbot_in_warehouse/sim/vector_description/urdf/vector.ros2_control.xacro (robot description, xacro)
@@ -97,4 +97,32 @@
       <state_interface name="velocity"/>
     </joint>
+    <joint name="torso_to_neck_1_joint">
+      <command_interface name="position"/>
+      <state_interface name="position">
+        <param name="initial_value">0.0</param>
+      </state_interface>
+      <state_interface name="velocity"/>
+    </joint>
+    <joint name="neck_1_to_neck_2_joint">
+      <command_interface name="position"/>
+      <state_interface name="position">
+        <param name="initial_value">0.0</param>
+      </state_interface>
+      <state_interface name="velocity"/>
+    </joint>
+    <joint name="left_wrist_1">
+      <command_interface name="position"/>
+      <state_interface name="position">
+        <param name="initial_value">0.0</param>
+      </state_interface>
+      <state_interface name="velocity"/>
+    </joint>
+    <joint name="left_wrist_2">
+      <command_interface name="position"/>
+      <state_interface name="position">
+        <param name="initial_value">0.0</param>
+      </state_interface>
+      <state_interface name="velocity"/>
+    </joint>
   </ros2_control>
 </robot>

File: vectorbot_in_warehouse/sim/vector_description/urdf/vector.xacro (robot description, xacro)
@@ -2873,5 +2873,358 @@
         </visual>
 <visual>
-            <origin xyz="-0.105326 0.066066 0.075423" rpy="-3.14159 3.3231e-15 -1.5708" />
+            <origin xyz="-0.085576 0.051366 -0.074326" rpy="0 -1.5708 1.5708" />
+            <geometry>
+                <mesh filename="file://$(find vector_description)/meshes/Part_3_Mirrored_Mirrored.stl" scale="1 1 1" />
+            </geometry>
+            <material name="0.972549_0.529412_0.003922_0.000000_0.000000">
+                <texture />
+                <color rgba="0.972549 0.529412 0.00392157 1" />
+            </material>
+        </visual>
+<visual>
+            <origin xyz="-0.271676 0.062366 0.030673" rpy="1.22465e-16 1.9475e-30 1.5708" />
+            <geometry>
+                <mesh filename="file://$(find vector_description)/meshes/L_S1_cover.stl" scale="1 1 1" />
+            </geometry>
+            <material name="0.917647_0.917647_0.917647_0.000000_0.000000">
+                <texture />
+                <color rgba="0.917647 0.917647 0.917647 1" />
+            </material>
+        </visual>
+<visual>
+            <origin xyz="-0.217176 0.030713 -0.028717" rpy="1.22465e-16 1.18329e-30 1.5708" />
+            <geometry>
+                <mesh filename="file://$(find vector_description)/meshes/L_S1_motor_bracket.stl" scale="1 1 1" />
+            </geometry>
+            <material name="0.647059_0.647059_0.647059_0.000000_0.000000">
+                <texture />
+                <color rgba="0.647059 0.647059 0.647059 1" />
+            </material>
+        </visual>
+<visual>
+            <origin xyz="-0.175676 0.145366 -0.044081" rpy="1.5708 6.12323e-17 -3.67761e-16" />
+            <geometry>
+                <mesh filename="file://$(find vector_description)/meshes/EVA_stp.stl" scale="1 1 1" />
+            </geometry>
+            <material name="0.792157_0.819608_0.933333_0.000000_0.000000">
+                <texture />
+                <color rgba="0.792157 0.819608 0.933333 1" />
+            </material>
+        </visual>
+<visual>
+            <origin xyz="-0.175676 0.145366 -0.044081" rpy="1.5708 6.12323e-17 -3.67761e-16" />
+            <geometry>
+                <mesh filename="file://$(find vector_description)/meshes/_5INCH_LCD_stp.stl" scale="1 1 1" />
+            </geometry>
+            <material name="0.792157_0.819608_0.933333_0.000000_0.000000">
+                <texture />
+                <color rgba="0.792157 0.819608 0.933333 1" />
+            </material>
+        </visual>
+<visual>
+            <origin xyz="-0.175676 0.145366 -0.044081" rpy="1.5708 6.12323e-17 -3.67761e-16" />
+            <geometry>
+                <mesh filename="file://$(find vector_description)/meshes/EVA_stp_1.stl" scale="1 1 1" />
+            </geometry>
+            <material name="0.792157_0.819608_0.933333_0.000000_0.000000">
+                <texture />
+                <color rgba="0.792157 0.819608 0.933333 1" />
+            </material>
+        </visual>
+<visual>
+            <origin xyz="-0.175676 0.145366 -0.044081" rpy="1.5708 6.12323e-17 -3.67761e-16" />
+            <geometry>
+                <mesh filename="file://$(find vector_description)/meshes/_5INCH_TP_stp.stl" scale="1 1 1" />
+            </geometry>
+            <material name="0.792157_0.819608_0.933333_0.000000_0.000000">
+                <texture />
+                <color rgba="0.792157 0.819608 0.933333 1" />
+            </material>
+        </visual>
+<visual>
+            <origin xyz="-0.175676 0.145366 -0.044081" rpy="1.5708 6.12323e-17 -3.67761e-16" />
+            <geometry>
+                <mesh filename="file://$(find vector_description)/meshes/EVA_stp_2.stl" scale="1 1 1" />
+            </geometry>
+            <material name="0.792157_0.819608_0.933333_0.000000_0.000000">
+                <texture />
+                <color rgba="0.792157 0.819608 0.933333 1" />
+            </material>
+        </visual>
+<visual>
+            <origin xyz="-0.170376 0.145816 0.087963" rpy="0 1.5708 -3.14159" />
+            <geometry>
+                <mesh filename="file://$(find vector_description)/meshes/USB_J4_10118194_606F1A_stp.stl" scale="1 1 1" />
+            </geometry>
+            <material name="0.615686_0.811765_0.929412_0.000000_0.000000">
+                <texture />
+                <color rgba="0.615686 0.811765 0.929412 1" />
+            </material>
+        </visual>
+<visual>
+            <origin xyz="-0.059576 0.145816 -0.102288" rpy="0 -1.5708 3.14159" />
+            <geometry>
+                <mesh filename="file://$(find vector_description)/meshes/USB_J4_10118194_606F1A_stp.stl" scale="1 1 1" />
+            </geometry>
+            <material name="0.615686_0.811765_0.929412_0.000000_0.000000">
+                <texture />
+                <color rgba="0.615686 0.811765 0.929412 1" />
+            </material>
+        </visual>
+<visual>
+            <origin xyz="-0.176176 0.141741 -0.004738" rpy="0 1.5708 -3.14159" />
+            <geometry>
+                <mesh filename="file://$(find vector_description)/meshes/HDMI_J1_47151_0001_61277A9B_stp.stl" scale="1 1 1" />
+            </geometry>
+            <material name="0.792157_0.819608_0.933333_0.000000_0.000000">
+                <texture />
+                <color rgba="0.792157 0.819608 0.933333 1" />
+            </material>
+        </visual>
+<visual>
+            <origin xyz="-0.054912 0.145266 0.015883" rpy="0 -1.5708 3.14159" />
+            <geometry>
+                <mesh filename="file://$(find vector_description)/meshes/SWITCH_7X3_3X3_5_stp.stl" scale="1 1 1" />
+            </geometry>
+            <material name="0.792157_0.819608_0.933333_0.000000_0.000000">
+                <texture />
+                <color rgba="0.792157 0.819608 0.933333 1" />
+            </material>
+        </visual>
+<visual>
+            <origin xyz="-0.054912 0.145266 -0.007383" rpy="0 -1.5708 3.14159" />
+            <geometry>
+                <mesh filename="file://$(find vector_description)/meshes/SWITCH_7X3_3X3_5_stp.stl" scale="1 1 1" />
+            </geometry>
+            <material name="0.792157_0.819608_0.933333_0.000000_0.000000">
+                <texture />
+                <color rgba="0.792157 0.819608 0.933333 1" />
+            </material>
+        </visual>
+<visual>
+            <origin xyz="-0.175676 0.145366 -0.044081" rpy="1.5708 6.12323e-17 -3.67761e-16" />
+            <geometry>
+                <mesh filename="file://$(find vector_description)/meshes/RTD2660_5INCH_HDMI_PCBA_stp.stl" scale="1 1 1" />
+            </geometry>
+            <material name="0.792157_0.819608_0.933333_0.000000_0.000000">
+                <texture />
+                <color rgba="0.792157 0.819608 0.933333 1" />
+            </material>
+        </visual>
+<visual>
+            <origin xyz="-0.137617 0.139366 0.031373" rpy="0 -1.5708 1.5708" />
+            <geometry>
+                <mesh filename="file://$(find vector_description)/meshes/HP2_0_4PIN_SMT_00_stp.stl" scale="1 1 1" />
+            </geometry>
+            <material name="0.792157_0.819608_0.933333_0.000000_0.000000">
+                <texture />
+                <color rgba="0.792157 0.819608 0.933333 1" />
+            </material>
+        </visual>
+<visual>
+            <origin xyz="-0.175672 0.145171 -0.026288" rpy="0 -1.5708 3.14159" />
+            <geometry>
+                <mesh filename="file://$(find vector_description)/meshes/MINI_HDMI_stp.stl" scale="1 1 1" />
+            </geometry>
+            <material name="0.792157_0.819608_0.933333_0.000000_0.000000">
+                <texture />
+                <color rgba="0.792157 0.819608 0.933333 1" />
+            </material>
+        </visual>
+<visual>
+            <origin xyz="-0.175676 0.145366 -0.044081" rpy="1.5708 6.12323e-17 -3.67761e-16" />
+            <geometry>
+                <mesh filename="file://$(find vector_description)/meshes/RTD2660_5INCH_HDMI_PCBA_stp_1.stl" scale="1 1 1" />
+            </geometry>
+            <material name="0.792157_0.819608_0.933333_0.000000_0.000000">
+                <texture />
+                <color rgba="0.792157 0.819608 0.933333 1" />
+            </material>
+        </visual>
+<visual>
+            <origin xyz="-0.175676 0.145366 -0.044081" rpy="1.5708 6.12323e-17 -3.67761e-16" />
+            <geometry>
+                <mesh filename="file://$(find vector_description)/meshes/_30PIN_CONNECTOR_stp.stl" scale="1 1 1" />
+            </geometry>
+            <material name="0.792157_0.819608_0.933333_0.000000_0.000000">
+                <texture />
+                <color rgba="0.792157 0.819608 0.933333 1" />
+            </material>
+        </visual>
+<visual>
+            <origin xyz="-0.175672 0.145171 -0.026288" rpy="0 -1.5708 3.14159" />
+            <geometry>
+                <mesh filename="file://$(find vector_description)/meshes/MINI_HDMI_stp_1.stl" scale="1 1 1" />
+            </geometry>
+            <material name="0.792157_0.819608_0.933333_0.000000_0.000000">
+                <texture />
+                <color rgba="0.792157 0.819608 0.933333 1" />
+            </material>
+        </visual>
+<visual>
+            <origin xyz="-0.054912 0.145266 0.027513" rpy="0 -1.5708 3.14159" />
+            <geometry>
+                <mesh filename="file://$(find vector_description)/meshes/SWITCH_7X3_3X3_5_stp.stl" scale="1 1 1" />
+            </geometry>
+            <material name="0.792157_0.819608_0.933333_0.000000_0.000000">
+                <texture />
+                <color rgba="0.792157 0.819608 0.933333 1" />
+            </material>
+        </visual>
+<visual>
+            <origin xyz="-0.175676 0.145366 -0.044081" rpy="1.5708 6.12323e-17 -3.67761e-16" />
+            <geometry>
+                <mesh filename="file://$(find vector_description)/meshes/_6PIN_CONNECTOR_stp.stl" scale="1 1 1" />
+            </geometry>
+            <material name="0.792157_0.819608_0.933333_0.000000_0.000000">
+                <texture />
+                <color rgba="0.792157 0.819608 0.933333 1" />
+            </material>
+        </visual>
+<visual>
+            <origin xyz="-0.175672 0.145171 -0.026288" rpy="0 -1.5708 3.14159" />
+            <geometry>
+                <mesh filename="file://$(find vector_description)/meshes/MINI_HDMI_stp_2.stl" scale="1 1 1" />
+            </geometry>
+            <material name="0.792157_0.819608_0.933333_0.000000_0.000000">
+                <texture />
+                <color rgba="0.792157 0.819608 0.933333 1" />
+            </material>
+        </visual>
+<visual>
+            <origin xyz="-0.175676 0.145366 -0.044081" rpy="1.5708 6.12323e-17 -3.67761e-16" />
+            <geometry>
+                <mesh filename="file://$(find vector_description)/meshes/HP_stp.stl" scale="1 1 1" />
+            </geometry>
+            <material name="0.792157_0.819608_0.933333_0.000000_0.000000">
+                <texture />
+                <color rgba="0.792157 0.819608 0.933333 1" />
+            </material>
+        </visual>
+<visual>
+            <origin xyz="-0.175672 0.145171 -0.026288" rpy="0 -1.5708 3.14159" />
+            <geometry>
+                <mesh filename="file://$(find vector_description)/meshes/MINI_HDMI_stp_3.stl" scale="1 1 1" />
+            </geometry>
+            <material name="0.792157_0.819608_0.933333_0.000000_0.000000">
+                <texture />
+                <color rgba="0.792157 0.819608 0.933333 1" />
+            </material>
+        </visual>
+<visual>
+            <origin xyz="-0.054912 0.145266 0.004250" rpy="0 -1.5708 3.14159" />
+            <geometry>
+                <mesh filename="file://$(find vector_description)/meshes/SWITCH_7X3_3X3_5_stp.stl" scale="1 1 1" />
+            </geometry>
+            <material name="0.792157_0.819608_0.933333_0.000000_0.000000">
+                <texture />
+                <color rgba="0.792157 0.819608 0.933333 1" />
+            </material>
+        </visual>
+<visual>
+            <origin xyz="-0.054912 0.145266 -0.019017" rpy="0 -1.5708 3.14159" />
+            <geometry>
+                <mesh filename="file://$(find vector_description)/meshes/SWITCH_7X3_3X3_5_stp.stl" scale="1 1 1" />
+            </geometry>
+            <material name="0.792157_0.819608_0.933333_0.000000_0.000000">
+                <texture />
+                <color rgba="0.792157 0.819608 0.933333 1" />
+            </material>
+        </visual>
+<visual>
+            <origin xyz="-0.175676 0.145366 -0.044081" rpy="1.5708 6.12323e-17 -3.67761e-16" />
+            <geometry>
+                <mesh filename="file://$(find vector_description)/meshes/RTD2660_5INCH_HDMI_PCBA_stp_2.stl" scale="1 1 1" />
+            </geometry>
+            <material name="0.792157_0.819608_0.933333_0.000000_0.000000">
+                <texture />
+                <color rgba="0.792157 0.819608 0.933333 1" />
+            </material>
+        </visual>
+        <visual>
+            <origin xyz="-0.115176 -0.0361336 -0.015826" rpy="0 1.5708 -1.2326e-32" />
+            <geometry>
+                <mesh filename="file://$(find vector_description)/meshes/HGH20CA1R1000Z0C_GW2025030058_6.stl" scale="1 1 1" />
+            </geometry>
+            <material name="0.231373_0.380392_0.705882_0.000000_0.000000">
+                <texture />
+                <color rgba="0.231373 0.380392 0.705882 1" />
+            </material>
+        </visual>
+        <visual>
+            <origin xyz="-0.115176 -0.0361336 -0.015826" rpy="0 1.5708 -1.2326e-32" />
+            <geometry>
+                <mesh filename="file://$(find vector_description)/meshes/HGH20CA1R1000Z0C_GW2025030058_5.stl" scale="1 1 1" />
+            </geometry>
+            <material name="0.917647_0.917647_0.917647_0.000000_0.000000">
+                <texture />
+                <color rgba="0.917647 0.917647 0.917647 1" />
+            </material>
+        </visual>
+        <visual>
+            <origin xyz="-0.115176 -0.0361336 -0.015826" rpy="0 1.5708 -1.2326e-32" />
+            <geometry>
+                <mesh filename="file://$(find vector_description)/meshes/HGH20CA1R1000Z0C_GW2025030058_7.stl" scale="1 1 1" />
+            </geometry>
+            <material name="0.647059_0.647059_0.647059_0.000000_0.000000">
+                <texture />
+                <color rgba="0.647059 0.647059 0.647059 1" />
+            </material>
+        </visual>
+        <visual>
+            <origin xyz="-0.115176 -0.0361336 -0.015826" rpy="0 1.5708 -1.2326e-32" />
+            <geometry>
+                <mesh filename="file://$(find vector_description)/meshes/HGH20CA1R1000Z0C_GW2025030058_3.stl" scale="1 1 1" />
+            </geometry>
+            <material name="0.972549_0.529412_0.003922_0.000000_0.000000">
+                <texture />
+                <color rgba="0.972549 0.529412 0.00392157 1" />
+            </material>
+        </visual>
+</link>
+    <!-- neck_link_1: Neck-bracket and Neck-bracket-support-3dprinted split from torso_link -->
+    <link name="neck_link_1">
+        <inertial>
+            <mass value="0.15" />
+            <origin xyz="0 0 0" rpy="0 0 0" />
+            <inertia ixx="1.0e-04" ixy="0.0" ixz="0.0" iyy="1.0e-04" iyz="0.0" izz="1.0e-04" />
+        </inertial>
+        <visual>
+            <origin xyz="0 0 0" rpy="1.23793e-28 -6.12323e-17 -3.14159" />
+            <geometry>
+                <mesh filename="file://$(find vector_description)/meshes/Neck_bracket_support_3dprinted.stl" scale="1 1 1" />
+            </geometry>
+            <material name="0.647059_0.647059_0.647059_0.000000_0.000000">
+                <texture />
+                <color rgba="0.647059 0.647059 0.647059 1" />
+            </material>
+        </visual>
+        <visual>
+            <origin xyz="0 0 0" rpy="1.24605e-28 -6.12323e-17 -3.14159" />
+            <geometry>
+                <mesh filename="file://$(find vector_description)/meshes/Neck_bracket.stl" scale="1 1 1" />
+            </geometry>
+            <material name="0.917647_0.917647_0.917647_0.000000_0.000000">
+                <texture />
+                <color rgba="0.917647 0.917647 0.917647 1" />
+            </material>
+        </visual>
+    </link>
+    <joint name="torso_to_neck_1_joint" type="revolute">
+        <origin xyz="-0.115176 0.058366 0.108173" rpy="0 0 0" />
+        <axis xyz="0 0 1" />
+        <parent link="torso_link" />
+        <child link="neck_link_1" />
+        <limit lower="-1.5708" upper="1.5708" effort="50.0" velocity="3.0" />
+    </joint>
+    <!-- neck_link_2: WEBCAM-Final-Assembly-Neck-Mechanism parts split from torso_link -->
+    <link name="neck_link_2">
+        <inertial>
+            <mass value="0.25" />
+            <origin xyz="0.115326 -0.055066 -0.049673" rpy="0 0 0" />
+            <inertia ixx="2.0e-04" ixy="0.0" ixz="0.0" iyy="2.0e-04" iyz="0.0" izz="2.0e-04" />
+        </inertial>
+<visual>
+            <origin xyz="0.01 0.011 0.02575" rpy="-3.14159 3.3231e-15 -1.5708" />
             <geometry>
                 <mesh filename="file://$(find vector_description)/meshes/eBom_FreeParts.stl" scale="1 1 1" />
@@ -2883,5 +3236,5 @@
         </visual>
 <visual>
-            <origin xyz="-0.105326 0.066066 0.075423" rpy="-3.14159 3.3231e-15 -1.5708" />
+            <origin xyz="0.01 0.011 0.02575" rpy="-3.14159 3.3231e-15 -1.5708" />
             <geometry>
                 <mesh filename="file://$(find vector_description)/meshes/eBom_FreeParts_1.stl" scale="1 1 1" />
@@ -2893,5 +3246,5 @@
         </visual>
 <visual>
-            <origin xyz="-0.115326 0.055066 0.049673" rpy="1.5708 -5.10703e-15 -1.5708" />
+            <origin xyz="0 0 0" rpy="1.5708 -5.10703e-15 -1.5708" />
             <geometry>
                 <mesh filename="file://$(find vector_description)/meshes/Wheel_25kg.stl" scale="1 1 1" />
@@ -2903,5 +3256,5 @@
         </visual>
 <visual>
-            <origin xyz="-0.115326 0.055066 0.049673" rpy="-3.14159 3.3231e-15 -1.5708" />
+            <origin xyz="0 0 0" rpy="-3.14159 3.3231e-15 -1.5708" />
             <geometry>
                 <mesh filename="file://$(find vector_description)/meshes/_93475A210.stl" scale="1 1 1" />
@@ -2913,5 +3266,5 @@
         </visual>
 <visual>
-            <origin xyz="-0.115326 0.055075 0.101473" rpy="-3.14159 3.3231e-15 -1.5708" />
+            <origin xyz="0 0.000009 0.0518" rpy="-3.14159 3.3231e-15 -1.5708" />
             <geometry>
                 <mesh filename="file://$(find vector_description)/meshes/Gear__25R_0_00_.stl" scale="1 1 1" />
@@ -2923,5 +3276,5 @@
         </visual>
 <visual>
-            <origin xyz="-0.115326 0.055075 0.102573" rpy="-1.5708 -4.44089e-15 -1.5708" />
+            <origin xyz="0 0.000009 0.0529" rpy="-1.5708 -4.44089e-15 -1.5708" />
             <geometry>
                 <mesh filename="file://$(find vector_description)/meshes/Wheel_gear_25kg.stl" scale="1 1 1" />
@@ -2933,5 +3286,5 @@
         </visual>
 <visual>
-            <origin xyz="-0.115326 0.055066 0.049673" rpy="-3.14159 3.3231e-15 -1.5708" />
+            <origin xyz="0 0 0" rpy="-3.14159 3.3231e-15 -1.5708" />
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